File: Circuitos-atvd.kicad_pcb (KiCad board)
At the start: 2 copper layers, 21 parts, among them X2 32MHz

Commit message: adicionando correcoes
Parts:
- removed U2: ~, Package_DFN_QFN:QFN-28-1EP_6x6mm_P0.65mm_EP4.25x4.25mm_ThermalVias
- added U1: ~, Package_DFN_QFN:QFN-48-1EP_6x6mm_P0.4mm_EP4.2x4.2mm_ThermalVias, F.Cu at (150.7, 105.5)
- FB1: footprint Ferrite_THT:LairdTech_28C0236-0JW-10 -> Resistor_SMD:R_0201_0603Metric
- moved L2 51.0 mm to (123.5, 107.5)
- moved R1 46.2 mm to (123.7, 112.8)
- moved C6 37.2 mm to (117.0, 112.8)
- moved C7 37.2 mm to (117.2, 114.5)
- moved L1 36.3 mm to (134.2, 103.0)
- moved C10 33.6 mm to (120.1, 109.3)
- moved C11 33.6 mm to (120.1, 111.0)
- moved C12 33.6 mm to (120.1, 112.8)
- moved C13 33.6 mm to (120.1, 114.5)
- moved FB1 32.7 mm to (123.7, 105.5)
- moved L3 31.7 mm to (123.5, 109.3)
- moved L4 31.7 mm to (123.7, 111.0)
- moved C4 29.8 mm to (117.0, 109.3)
- moved C2 29.8 mm to (117.0, 107.5)
- moved C5 29.8 mm to (117.0, 111.0)
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Connections:
- net Earth renamed GND
